File: Schematic/Schematic.kicad_sch (KiCad schematic)
At the start: 17 parts, among them J3 FTDI, SW1 SW_Push, U1 ATmega328P-A, Y1 16 Mhz

Commit message: error PCB done 12 warning to do
Parts:
- C1, C2: symbol elec:Capacitor -> Elec_Nigel:Capacitor_12_pF
- C3, C4, C7: symbol elec:Capacitor -> Elec_Nigel:Capacitor_100nF
- C6: symbol elec:Capacitor -> Elec_Nigel:Capacitor_1uF
- D1: symbol elec:Led -> Elec_Nigel:Led_green
- D2: symbol elec:Led -> Elec_Nigel:Led_red
- J1: symbol elec:J1 -> Elec_Nigel:J1
- J2: symbol elec:j2 -> Elec_Nigel:j2
- J3: symbol elec:FTDI -> Elec_Nigel:FTDI
- R1: symbol elec:Resistor -> Elec_Nigel:Resistor_330
- R2, R3: symbol elec:Resistor -> Elec_Nigel:Resistor_10K
- SW1: symbol elec:Interrupteurs -> Elec_Nigel:Interrupteurs
- U1: symbol elec:Atmega328P -> Elec_Nigel:Atmega328P
- Y1: symbol elec:Oscillator -> Elec_Nigel:Oscillator
Changed lines of the file:
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@@
 	(wire
 		(pts
-			(xy 207.01 59.69) (xy 203.2 59.69)
+			(xy 203.2 59.69) (xy 207.01 59.69)
 		)
 		(stroke
@@
 	(wire
 		(pts
-			(xy 203.2 59.69) (xy 203.2 63.5)
+			(xy 81.28 40.64) (xy 81.28 41.91)
 		)
 		(stroke
@@
 	(wire
 		(pts
-			(xy 81.28 40.64) (xy 81.28 41.91)
+			(xy 114.3 118.11) (xy 123.19 118.11)
 		)
 		(stroke
@@
 	(wire
 		(pts
-			(xy 114.3 118.11) (xy 123.19 118.11)
+			(xy 26.67 102.87) (xy 26.67 105.41)
 		)
 		(stroke
@@
 	(wire
 		(pts
-			(xy 26.67 102.87) (xy 26.67 105.41)
+			(xy 105.41 118.11) (xy 107.95 118.11)
 		)
 		(stroke
@@
 	(wire
 		(pts
-			(xy 105.41 118.11) (xy 107.95 118.11)
+			(xy 203.2 63.5) (xy 203.2 59.69)
 		)
 		(stroke
@@
 	)
 	(symbol
-		(lib_id "elec:Capacitor")
+		(lib_id "Elec_Nigel:Capacitor_100nF")
 		(at 68.58 54.61 0)
 		(unit 1)
@@
 		)
 		(property "Footprint" "Library:SMD_603"
-			(at 68.58 54.61 0)
+			(at 64.516 60.452 0)
 			(effects
 				(font
@@
 		)
 		(property "Datasheet" "https://yageogroup.com/content/datasheet/asset/file/UPY-GPHC_X7R_6_3V-TO-250V"
-			(at 68.58 54.61 0)
+			(at 71.374 62.738 0)
 			(effects
 				(font
@@
 	)
 	(symbol
-		(lib_id "elec:GND")
+		(lib_id "Elec_Nigel:GND")
 		(at 95.25 146.05 0)
 		(unit 1)
@@
 	)
 	(symbol
-		(lib_id "elec:Capacitor")
+		(lib_id "Elec_Nigel:Capacitor_100nF")
 		(at 26.67 107.95 0)
 		(unit 1)
@@
 		)
 		(property "Footprint" "Library:SMD_603"
-			(at 26.67 107.95 0)
+			(at 22.606 113.792 0)
 			(effects
 				(font
@@
 		)
 		(property "Datasheet" "https://yageogroup.com/content/datasheet/asset/file/UPY-GPHC_X7R_6_3V-TO-250V"
-			(at 26.67 107.95 0)
+			(at 29.464 116.078 0)
 			(effects
 				(font
@@
 	)
 	(symbol
-		(lib_id "elec:Capacitor")
+		(lib_id "Elec_Nigel:Capacitor_1uF")
 		(at 48.26 54.61 0)
 		(unit 1)
@@
 	)
 	(symbol
-		(lib_id "elec:Atmega328P")
+		(lib_id "Elec_Nigel:Atmega328P")
 		(at 55.88 144.78 0)
 		(unit 1)
@@
 	)
 	(symbol
-		(lib_id "elec:Led")
+		(lib_id "Elec_Nigel:Led_green")
 		(at 148.59 48.26 0)
 		(unit 1)
@@
 	)
 	(symbol
-		(lib_id "elec:FTDI")
+		(lib_id "Elec_Nigel:FTDI")
 		(at 231.14 140.97 0)
 		(unit 1)
@@
 	)
 	(symbol
-		(lib_id "elec:VCC")
+		(lib_id "Elec_Nigel:VCC")
 		(at 55.88 97.79 0)
 		(unit 1)
@@
 	)
 	(symbol
-		(lib_id "elec:GND")
+		(lib_id "Elec_Nigel:GND")
 		(at 148.59 58.42 0)
 		(unit 1)
@@
 	)
 	(symbol
-		(lib_id "elec:GND")
+		(lib_id "Elec_Nigel:GND")
 		(at 48.26 66.04 0)
 		(unit 1)
@@
 	)
 	(symbol
-		(lib_id "elec:GND")
+		(lib_id "Elec_Nigel:GND")
 		(at 54.61 194.31 0)
 		(unit 1)
@@
 	)
 	(symbol
-		(lib_id "elec:Oscillator")
+		(lib_id "Elec_Nigel:Oscillator")
 		(at 105.41 130.81 0)
 		(unit 1)
@@
 	)
 	(symbol
-		(lib_id "elec:j2")
+		(lib_id "Elec_Nigel:j2")
 		(at 204.47 140.97 0)
 		(unit 1)
@@
 	)
 	(symbol
-		(lib_id "elec:VCC")
+		(lib_id "Elec_Nigel:VCC")
 		(at 81.28 35.56 0)
 		(unit 1)
@@
 	)
 	(symbol
-		(lib_id "elec:Capacitor")
+		(lib_id "Elec_Nigel:Capacitor_12_pF")
 		(at 110.49 118.11 90)
 		(unit 1)
@@
 	)
 	(symbol
-		(lib_id "elec:Capacitor")
+		(lib_id "Elec_Nigel:Capacitor_12_pF")
 		(at 110.49 149.86 90)
 		(unit 1)
@@
 	)
 	(symbol
-		(lib_id "power:PWR_FLAG")
+		(lib_id "Elec_Nigel:PWR_FLAG")
 		(at 81.28 68.58 270)
 		(unit 1)
@@
 	)
 	(symbol
-		(lib_id "elec:GND")
+		(lib_id "Elec_Nigel:GND")
 		(at 68.58 66.04 0)
 		(unit 1)
@@
 	)
 	(symbol
-		(lib_id "elec:Resistor")
+		(lib_id "Elec_Nigel:Resistor_330")
 		(at 148.59 31.75 0)
 		(unit 1)
@@
 	)
 	(symbol
-		(lib_id "elec:Led")
+		(lib_id "Elec_Nigel:Led_red")
 		(at 81.28 52.07 0)
 		(unit 1)
@@
 	)
 	(symbol
-		(lib_id "elec:GND")
+		(lib_id "Elec_Nigel:GND")
 		(at 81.28 74.93 0)
 		(unit 1)
@@
 	)
 	(symbol
-		(lib_id "elec:Resistor")
+		(lib_id "Elec_Nigel:Resistor_10K")
 		(at 81.28 60.96 0)
 		(unit 1)
@@
 	)
 	(symbol
-		(lib_id "elec:Capacitor")
+		(lib_id "Elec_Nigel:Capacitor_100nF")
 		(at 209.55 59.69 90)
 		(unit 1)
@@
 		)
 		(property "Footprint" "Library:SMD_603"
-			(at 209.55 59.69 0)
+			(at 215.392 63.754 0)
 			(effects
 				(font
@@
 		)
 		(property "Datasheet" "https://yageogroup.com/content/datasheet/asset/file/UPY-GPHC_X7R_6_3V-TO-250V"
-			(at 209.55 59.69 0)
+			(at 217.678 56.896 0)
 			(effects
 				(font
@@
 	)
 	(symbol
-		(lib_id "elec:GND")
+		(lib_id "Elec_Nigel:GND")
 		(at 130.81 146.05 0)
 		(unit 1)
@@
 	)
 	(symbol
-		(lib_id "elec:VCC")
+		(lib_id "Elec_Nigel:VCC")
 		(at 26.67 100.33 0)
 		(unit 1)
@@
 	)
 	(symbol
-		(lib_id "elec:VCC")
+		(lib_id "Elec_Nigel:VCC")
 		(at 234.95 40.64 0)
 		(unit 1)
@@
 	)
 	(symbol
-		(lib_id "elec:Interrupteurs")
+		(lib_id "Elec_Nigel:Interrupteurs")
 		(at 220.98 59.69 0)
 		(unit 1)
@@
 	)
 	(symbol
-		(lib_id "elec:J1")
+		(lib_id "Elec_Nigel:J1")
 		(at 160.02 139.7 0)
 		(unit 1)
@@
 	)
 	(symbol
-		(lib_id "elec:GND")
+		(lib_id "Elec_Nigel:GND")
 		(at 203.2 71.12 0)
 		(unit 1)
@@
 	)
 	(symbol
-		(lib_id "elec:Resistor")
+		(lib_id "Elec_Nigel:Resistor_10K")
 		(at 234.95 49.53 0)
 		(unit 1)
@@
 	)
 	(symbol
-		(lib_id "power:PWR_FLAG")
+		(lib_id "Elec_Nigel:PWR_FLAG")
 		(at 81.28 33.02 270)
 		(unit 1)

Commit message: pcb working
Connections:
- net RAW is gone; now on net VCC: C6.1, C7.1, D2.1, J2.1
- net RXO is gone; now on net TXO: U1.31 (PD1)
- net GND: now also C1.2, C2.2, C4.1, C6.2 (GND), C7.2, D1.2, R2.2, U1.3 (GND), Y1.2, Y1.4
- net VCC: now also C3.1, R3.1, U1.18 (AVCC), U1.4 (VCC)
Changed lines of the file:
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@@
 	)
 	(junction
+		(at 81.28 39.37)
+		(diameter 0)
+		(color 0 0 0 0)
+	)
+	(junction
+		(at 81.28 67.31)
+		(diameter 0)
+		(color 0 0 0 0)
+	)
+	(junction
 		(at 234.95 59.69)
 		(diameter 0)
@@
 	(wire
 		(pts
+			(xy 81.28 38.1) (xy 81.28 39.37)
+		)
+		(stroke
+			(width 0)
+			(type default)
+		)
+	)
+	(wire
+		(pts
 			(xy 86.36 149.86) (xy 105.41 149.86)
 		)
@@
 	(wire
 		(pts
-			(xy 114.3 118.11) (xy 123.19 118.11)
+			(xy 234.95 41.91) (xy 234.95 43.18)
 		)
 		(stroke
@@
 	(wire
 		(pts
-			(xy 26.67 102.87) (xy 26.67 105.41)
+			(xy 114.3 118.11) (xy 123.19 118.11)
 		)
 		(stroke
@@
 	(wire
 		(pts
-			(xy 81.28 38.1) (xy 81.28 40.64)
+			(xy 81.28 39.37) (xy 81.28 40.64)
 		)
 		(stroke
@@
 	(wire
 		(pts
+			(xy 26.67 102.87) (xy 26.67 105.41)
+		)
+		(stroke
+			(width 0)
+			(type default)
+		)
+	)
+	(wire
+		(pts
 			(xy 123.19 130.81) (xy 123.19 149.86)
 		)
@@
 		)
 	)
-	(global_label "RXO"
+	(global_label "TXO"
 		(shape input)
 		(at 74.93 160.02 0)
@@
 		)
 		(property "Intersheetrefs" "${INTERSHEET_REFS}"
-			(at 81.7252 160.02 0)
+			(at 81.4228 160.02 0)
 			(effects
 				(font
@@
 			)
 		)
+		(property "VCC" ""
+			(at 41.91 42.8308 0)
+			(effects
+				(font
+					(size 1.27 1.27)
+				)
+				(justify right)
+				(hide yes)
+			)
+		)
 	)
 	(global_label "GND"
@@
 	)
 	(symbol
+		(lib_id "Elec_Nigel:PWR_FLAG_INPUT")
+		(at 81.28 39.37 270)
+		(unit 1)
+		(exclude_from_sim no)
+		(in_bom yes)
+		(on_board yes)
+		(dnp no)
+		(fields_autoplaced yes)
+		(property "Reference" "#FLG03"
+			(at 87.884 28.702 0)
+			(effects
+				(font
+					(size 1.27 1.27)
+				)
+				(hide yes)
+			)
+		)
+		(property "Value" "PWR_FLAG_INPUT"
+			(at 85.09 39.3699 90)
+			(effects
+				(font
+					(size 1.27 1.27)
+				)
+				(justify left)
+			)
+		)
+		(property "Footprint" ""
+			(at 81.28 39.37 0)
+			(effects
+				(font
+					(size 1.27 1.27)
+				)
+				(hide yes)
+			)
+		)
+		(property "Datasheet" "~"
+			(at 81.28 39.37 0)
+			(effects
+				(font
+					(size 1.27 1.27)
+				)
+				(hide yes)
+			)
+		)
+		(property "Description" "Special symbol for telling ERC where power comes from"
+			(at 77.216 39.116 0)
+			(effects
+				(font
+					(size 1.27 1.27)
+				)
+				(hide yes)
+			)
+		)
+		(pin "1"
+		)
+		(instances
+			(project "Schematic"
+				(path "/a7fd653e-c1fb-497b-80dc-689b3cc1b28c"
+					(reference "#FLG03")
+					(unit 1)
+				)
+			)
+		)
+	)
+	(symbol
 		(lib_id "Elec_Nigel:VCC")
 		(at 55.88 97.79 0)
@@
 		(dnp no)
 		(property "Reference" "#PWR3"
-			(at 53.848 86.106 0)
+			(at 57.404 93.472 0)
 			(do_not_autoplace yes)
 			(effects
@@
 		(on_board yes)
 		(dnp no)
-		(property "Reference" "#PWR1"
+		(property "Reference" "#PWD0101"
 			(at 45.974 68.326 0)
 			(effects
@@
 			(project "Schematic"
 				(path "/a7fd653e-c1fb-497b-80dc-689b3cc1b28c"
-					(reference "#PWR1")
+					(reference "#PWD0101")
 					(unit 1)
 				)
@@
 	)
 	(symbol
-		(lib_id "Elec_Nigel:PWR_FLAG")
-		(at 81.28 68.58 270)
+		(lib_id "Elec_Nigel:PWR_FLAG_OUTPUT")
+		(at 81.28 67.31 270)
 		(unit 1)
 		(exclude_from_sim no)
@@
 		(fields_autoplaced yes)
 		(property "Reference" "#FLG02"
-			(at 83.185 68.58 0)
+			(at 87.884 56.642 0)
 			(effects
 				(font
@@
 			)
 		)
-		(property "Value" "PWR_FLAG"
-			(at 85.09 68.5799 90)
+		(property "Value" "PWR_FLAG_OUTPUT"
+			(at 85.09 67.3099 90)
 			(effects
 				(font
@@
 		)
 		(property "Footprint" ""
-			(at 81.28 68.58 0)
+			(at 81.28 67.31 0)
 			(effects
 				(font
@@
 		)
 		(property "Datasheet" "~"
-			(at 81.28 68.58 0)
+			(at 81.28 67.31 0)
 			(effects
 				(font
@@
 		)
 		(property "Description" "Special symbol for telling ERC where power comes from"
-			(at 81.28 68.58 0)
+			(at 77.216 67.056 0)
 			(effects
 				(font
@@
 	(symbol
 		(lib_id "Elec_Nigel:VCC")
-		(at 234.95 40.64 0)
+		(at 234.95 39.37 0)
 		(unit 1)
 		(exclude_from_sim no)
@@
 		(dnp no)
 		(property "Reference" "#PWR11"
-			(at 238.76 34.2899 0)
+			(at 238.76 33.0199 0)
 			(effects
 				(font
@@
 		)
 		(property "Value" "VCC"
-			(at 233.172 28.448 0)
+			(at 233.172 27.178 0)
 			(effects
 				(font
@@
 		)
 		(property "Footprint" ""
-			(at 234.95 40.64 0)
+			(at 234.95 39.37 0)
 			(effects
 				(font
@@
 		)
 		(property "Datasheet" ""
-			(at 234.95 40.64 0)
+			(at 234.95 39.37 0)
 			(effects
 				(font
@@
 		)
 		(property "Description" ""
-			(at 234.95 40.64 0)
+			(at 234.95 39.37 0)
 			(effects
 				(font
@@
 					(unit 1)
 				)
-			)
-		)
-	)
-	(symbol
-		(lib_id "Elec_Nigel:PWR_FLAG")
-		(at 81.28 33.02 270)
-		(unit 1)
-		(exclude_from_sim no)
-		(in_bom yes)
-		(on_board yes)
-		(dnp no)
-		(fields_autoplaced yes)
-		(property "Reference" "#FLG01"
-			(at 83.185 33.02 0)
-			(effects
-				(font
-					(size 1.27 1.27)
-				)
-				(hide yes)
-			)
-		)
-		(property "Value" "PWR_FLAG"
-			(at 85.09 33.0199 90)
-			(effects
-				(font
-					(size 1.27 1.27)
-				)
-				(justify left)
-			)
-		)
-		(property "Footprint" ""
-			(at 81.28 33.02 0)
-			(effects
-				(font
-					(size 1.27 1.27)
-				)
-				(hide yes)
-			)
-		)
-		(property "Datasheet" "~"
-			(at 81.28 33.02 0)
-			(effects
-				(font
-					(size 1.27 1.27)
-				)
-				(hide yes)
-			)
-		)
-		(property "Description" "Special symbol for telling ERC where power comes from"
-			(at 81.28 33.02 0)
-			(effects
-				(font
-					(size 1.27 1.27)
-				)
-				(hide yes)
-			)
-		)
-		(pin "1"
-		)
-		(instances
-			(project "Schematic"
-				(path "/a7fd653e-c1fb-497b-80dc-689b3cc1b28c"
-					(reference "#FLG01")
-					(unit 1)
-				)

Commit message: updated board
Parts:
- SW1: footprint Library:Interrupter_SMD_Omron_B3S-1000 -> Library:interupter_SMD_B3U-1000P(M)
Changed lines of the file:
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@@
 			)
 		)
-		(property "Footprint" "Library:Interrupter_SMD_Omron_B3S-1000"
+		(property "Footprint" "Library:interupter_SMD_B3U-1000P(M)"
 			(at 220.98 59.69 0)
 			(effects
@@
 			)
 		)
-		(property "Datasheet" "https://octopart.com/datasheet/omron/B3S-1000"
+		(property "Datasheet" "https://omronfs.omron.com/en_US/ecb/products/pdf/en-b3u.pdf"
 			(at 220.98 59.69 0)
 			(effects
